File: Kicad/environment master/Environmental_monitoring_device.kicad_pcb (KiCad board)
At the start: 2 copper layers, 53.8 x 62.9 mm, 43 parts, among them J2 RS485 OUT, J3 RS485 OUT, J4 Conn_01x10, J5 Barrel_Jack_Switch_Pin3Ring, U1 RFM95W-868S2, U2 ESP32-C3-MINI-1U-N4, U3 MAX485E, U4 LM2596S-5, U5 AMS1117-3.3

Commit message: resolves issue #1
Parts:
- U3: value MAX485E -> THVD1406
- renumbered locked to J1
