File: Kicad/environment master/Environmental_monitoring_device.kicad_sch (KiCad schematic)
At the start: 40 parts, among them J1 Barrel_Jack_Switch_Pin3Ring, J2 U.FL-R-SMT_01_, J3 Conn_01x10, J4 RS485 OUT, J5 RS485 OUT, U1 ESP32-C3-MINI-1U-N4, U2 AMS1117-3.3, U3 RFM95W-868S2, U4 MAX485E, U5 LM2596S-5

Commit message: resolves issue #1
Parts:
- U4: value MAX485E -> THVD1406
Changed lines of the file:
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@@
 			)
 		)
-		(property "Value" "MAX485E"
+		(property "Value" "THVD1406"
 			(at 180.34 29.21 0)
 			(effects
@@
 			)
 		)
-		(property "Datasheet" "https://datasheets.maximintegrated.com/en/ds/MAX1487E-MAX491E.pdf"
+		(property "Datasheet" "https://www.ti.com/lit/ds/symlink/thvd1406.pdf?ts=1751614038517&ref_url=https%253A%252F%252Fwww.google.com%252F"
 			(at 179.07 39.37 0)
 			(effects
