File: Kicad/environment slave/environment slave.kicad_pcb (KiCad board)
At the start: 2 copper layers, 79.2 x 68.8 mm, 72 parts, among them J1 Barrel_Jack, J2 U.FL-R-SMT_01_, J3 Solar, J4 Conn_01x10, J5 PWR OUT, J6 USB_C_Receptacle_PowerOnly_6P, J7 RS485 OUT, U1 MIC5219-3.3v, U2 ESP32-C3-MINI-1U-N4, U3 RFM95W-868S2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

Commit message: resolves issue #1
Parts:
- U4: value MAX485E -> THVD1406
Changed lines of the file:
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@@
 			)
 		)
-		(property "Value" "MAX485E"
+		(property "Value" "THVD1406"
 			(at 0 4.05 0)
 			(layer "F.Fab")
@@
 			)
 		)
-		(property "Datasheet" ""
+		(property "Datasheet" "https://www.ti.com/lit/ds/symlink/thvd1406.pdf?ts=1751614038517&ref_url=https%253A%252F%252Fwww.google.com%252F"
 			(at 0 0 0)
 			(layer "F.Fab")
